File: TempCtrl.sch (KiCad schematic (older format))
At the start: 23 parts, among them P1 CONN_01X02, P2 CONN_01X05, Q1 BD678, U1 LM358

Commit message: Added PNG images
Parts:
- P1: value CONN_01X02 -> PWR 18-24V
Changed lines of the file:
@@
 P 1700 2200
 F 0 "P1" H 1700 2350 50  0000 C CNN
-F 1 "CONN_01X02" V 1800 2200 50  0000 C CNN
+F 1 "PWR 18-24V" V 1800 2200 50  0000 C CNN
 F 2 "Socket_Strips:Socket_Strip_Angled_1x02" H 1700 2200 50  0001 C CNN
 F 3 "" H 1700 2200 50  0000 C CNN
@@
 F 0 "Q1" H 6600 2925 50  0000 L CNN
 F 1 "BD678" H 6600 2850 50  0000 L CNN
-F 2 "TO_SOT_Packages_THT:SOT126_SOT32_Housing_Horizontal" H 6600 2775 50  0000 L CIN
+F 2 "TO_SOT_Packages_THT:SOT126_SOT32_Housing_Horizontal" H 6600 2775 50  0001 L CIN
 F 3 "" H 6350 2850 50  0000 L CNN
 	1    6350 2850

Commit message: Final version
Connections:
- net GNDREF: now also P2.1 (P1); no longer P2.3 (P3)
- net VCC: now also Q1.3 (E), R1.2; no longer Q1.2 (C), R1.1
- net at C2.1, R2.2, R3.2: now also P2.3 (P3); no longer P2.4 (P4)
- net at P2.5 (P5): now also Q1.2 (C), R13.2; no longer R1.2
- new net: P2.4 (P4), R1.1
Other:
- moved on the sheet: P2, R1
Changed lines of the file:
@@
 L GNDREF #PWR01
 U 1 1 5888B7E4
-P 6450 5000
-F 0 "#PWR01" H 6450 4750 50  0001 C CNN
-F 1 "GNDREF" H 6450 4850 50  0000 C CNN
-F 2 "" H 6450 5000 50  0000 C CNN
-F 3 "" H 6450 5000 50  0000 C CNN
-	1    6450 5000
-	1    0    0    -1
+P 6400 4550
+F 0 "#PWR01" H 6400 4300 50  0001 C CNN
+F 1 "GNDREF" V 6400 4250 50  0000 C CNN
+F 2 "" H 6400 4550 50  0000 C CNN
+F 3 "" H 6400 4550 50  0000 C CNN
+	1    6400 4550
+	0    1    1    0
 $EndComp
 $Comp
@@
 L CONN_01X05 P2
 U 1 1 58891446
-P 7000 4650
-F 0 "P2" H 7000 4950 50  0000 C CNN
-F 1 "CONN_01X05" V 7100 4650 50  0000 C CNN
-F 2 "Socket_Strips:Socket_Strip_Straight_1x05" H 7000 4650 50  0001 C CNN
-F 3 "" H 7000 4650 50  0000 C CNN
-	1    7000 4650
-	1    0    0    -1
-$EndComp
-Text Notes 7150 4500 0    60   ~ 0
+P 7150 4750
+F 0 "P2" H 7150 5050 50  0000 C CNN
+F 1 "CONN_01X05" V 7250 4750 50  0000 C CNN
+F 2 "Socket_Strips:Socket_Strip_Straight_1x05" H 7150 4750 50  0001 C CNN
+F 3 "" H 7150 4750 50  0000 C CNN
+	1    7150 4750
+	1    0    0    -1
+$EndComp
+Text Notes 7350 4600 0    60   ~ 0
 H1
-Text Notes 7150 4600 0    60   ~ 0
+Text Notes 7350 4700 0    60   ~ 0
 H2
-Text Notes 7150 4700 0    60   ~ 0
+Text Notes 7350 4800 0    60   ~ 0
 T1
-Text Notes 7150 4800 0    60   ~ 0
+Text Notes 7350 4900 0    60   ~ 0
 T2
-Text Notes 7150 4900 0    60   ~ 0
+Text Notes 7350 5000 0    60   ~ 0
 ESD\n
 $Comp
@@
 F 3 "" H 6350 2850 50  0000 L CNN
 	1    6350 2850
-	1    0    0    -1
+	1    0    0    1
 $EndComp
 $Comp
 L PWR_FLAG #FLG03
 U 1 1 588DC5FB
-P 2550 2150
-F 0 "#FLG03" H 2550 2245 50  0001 C CNN
-F 1 "PWR_FLAG" H 2550 2330 50  0000 C CNN
-F 2 "" H 2550 2150 50  0000 C CNN
-F 3 "" H 2550 2150 50  0000 C CNN
-	1    2550 2150
+P 2300 2150
+F 0 "#FLG03" H 2300 2245 50  0001 C CNN
+F 1 "PWR_FLAG" H 2300 2330 50  0000 C CNN
+F 2 "" H 2300 2150 50  0000 C CNN
+F 3 "" H 2300 2150 50  0000 C CNN
+	1    2300 2150
 	1    0    0    -1
 $EndComp
@@
 L R R1
 U 1 1 588A1762
-P 2550 4200
-F 0 "R1" V 2630 4200 50  0000 C CNN
-F 1 "1K" V 2550 4200 50  0000 C CNN
-F 2 "Resistors_SMD:R_0805" V 2480 4200 50  0001 C CNN
-F 3 "" H 2550 4200 50  0000 C CNN
-	1    2550 4200
-	1    0    0    -1
+P 6650 2150
+F 0 "R1" V 6730 2150 50  0000 C CNN
+F 1 "1K" V 6650 2150 50  0000 C CNN
+F 2 "Resistors_SMD:R_0805" V 6580 2150 50  0001 C CNN
+F 3 "" H 6650 2150 50  0000 C CNN
+	1    6650 2150
+	0    1    1    0
 $EndComp
 $Comp
@@
 	4800 2500 4750 2500
 Wire Wire Line
-	1900 2150 6450 2150
+	1900 2150 6500 2150
 Wire Wire Line
 	5100 2500 5600 2500
@@
 Wire Wire Line
 	1900 2250 1900 2700
-Wire Wire Line
-	2550 4350 2550 4850
-Wire Wire Line
-	2550 2150 2550 4050
 Wire Wire Line
 	6450 3550 6450 3500
@@
 Wire Wire Line
 	3550 2050 3550 2450
-Wire Wire Line
-	6450 3100 6800 3100
 $Comp
 L R R12
@@
 Connection ~ 6050 2850
 Connection ~ 6050 2150
-Wire Wire Line
-	6450 3950 6450 5000
 Connection ~ 6450 4650
-Wire Wire Line
-	6800 3100 6800 4450
 Connection ~ 1900 2250
 Wire Wire Line
-	2550 4850 6800 4850
-Wire Wire Line
-	3150 4650 6800 4650
-Wire Wire Line
-	6800 4550 6450 4550
+	3150 4650 6950 4650
+Wire Wire Line
+	6400 4550 6950 4550
 Connection ~ 6450 4550
 Wire Wire Line
-	2900 4750 6800 4750
-Connection ~ 2550 2150
+	2900 4750 6950 4750
 Wire Wire Line
 	1900 2600 2300 2600
@@
 	2300 2250 2300 2150
 Connection ~ 2300 2150
+Wire Wire Line
+	6450 3100 6600 3100
+Wire Wire Line
+	6600 3100 6600 4950
+Wire Wire Line
+	6800 2150 6800 4850
+Connection ~ 6450 2150
+Wire Wire Line
+	6450 3950 6450 4650
+Wire Wire Line
+	6800 4850 6950 4850
+Wire Wire Line
+	6600 4950 6950 4950
 $EndSCHEMATC
